File: PCB/EasyInjection.sch (KiCad schematic (older format))
At the start: 4 parts

Commit message: Version 1.0 done!
Parts:
- added J1: Conn_02x05_Top_Bottom, Connectors_Molex:Molex_MiniFit-JR-5569-10A1_2x05x4.20mm_Angled, symbol Conn_02x05_Top_Bottom
- added R1, R2, R5, R6: 1k, VND5N07:R_Axial_DIN0204_L3.6mm_D1.6mm_P7.62mm_Horizontal, symbol R
- added R3, R4, R7, R8: 100k, VND5N07:R_Axial_DIN0204_L3.6mm_D1.6mm_P7.62mm_Horizontal, symbol R
- S1, S2, S3, S4: value VND5N07-E -> VND5N07; footprint VND5N07-E:TO-252-(DPAK)_1 -> VND5N07:VND5N07_TO-252-(DPAK)
Connections:
- net at S1.1 (G): now also R1.1, R3.1
- net OUT_1: now reaches S1.2 (D)
- net OUT_1: now also J1.6 (Pin_6)
- net GNDPWR: now reaches S1.3 (S)
- net GNDPWR: now also S2.3 (S), S3.3 (S), S4.3 (S), J1.3 (Pin_3), J1.8 (Pin_8), R3.2, R4.2, R7.2, R8.2
- net at S3.1 (G): now also R5.1, R7.1
- net OUT_3: now reaches S3.2 (D)
- net OUT_3: now also J1.9 (Pin_9)
- net at S2.1 (G): now also R2.1, R4.1
- net OUT_2: now reaches S2.2 (D)
- net OUT_2: now also J1.7 (Pin_7)
- net at S4.1 (G): now also R6.1, R8.1
- net OUT_4: now reaches S4.2 (D)
- net OUT_4: now also J1.10 (Pin_10)
- new net CTRL_1: J1.2 (Pin_2), R1.2
- new net CTRL_2: J1.1 (Pin_1), R2.2
- new net CTRL_3: J1.5 (Pin_5), R5.2
- new net CTRL_4: J1.4 (Pin_4), R6.2
- no-connect marks 0 -> 1
Other:
- moved on the sheet: S1, S2, S3, S4

Commit message: Changed to 5 channels
Parts:
- removed J1: Conn_02x05_Top_Bottom, Connectors_Molex:Molex_MiniFit-JR-5569-10A1_2x05x4.20mm_Angled, symbol Conn_02x05_Top_Bottom
- added J1: Conn_02x06_Top_Bottom, Connector_Molex:Molex_Mini-Fit_Jr_5566-12A_2x06_P4.20mm_Vertical, symbol Connector_Generic:Conn_02x06_Top_Bottom
- added R5: 1k, VND5N07:R_Axial_DIN0204_L3.6mm_D1.6mm_P7.62mm_Horizontal, symbol EasyInjection-rescue:R
- added R6: 100k, VND5N07:R_Axial_DIN0204_L3.6mm_D1.6mm_P7.62mm_Horizontal, symbol EasyInjection-rescue:R
- added S5: VND5N07, VND5N07:VND5N07_TO-252-(DPAK), symbol EasyInjection-rescue:VND5N07-E
- R1, R4, R8: symbol R -> EasyInjection-rescue:R
- R10: renamed from R7; symbol R -> EasyInjection-rescue:R
- R2: renamed from R3; symbol R -> EasyInjection-rescue:R
- R3: renamed from R2; symbol R -> EasyInjection-rescue:R
- R7: renamed from R6; symbol R -> EasyInjection-rescue:R
- R9: renamed from R5; symbol R -> EasyInjection-rescue:R
- S1, S2, S3, S4: symbol VND5N07-E -> EasyInjection-rescue:VND5N07-E
Connections:
- net labels added: CTRL_5, OUT_5
- wire segments 37 -> 52
Other:
- moved on the sheet: R1, R10, R2, R3, R4, R7, R8, R9, S1, S2, S3, S4
